File: kicad/bass_compressor/bass_compressor.kicad_sch (KiCad schematic)
At the start: 47 parts, among them IC1 LM13700, IC3 TC4013BP, J1 6.3mm TRS(mono use), J2 6.3mm TS(out), Q1 2SC1815, Q2 2SC1815, SW1 Cherry MX (手持ち), U1 TL072

Commit message: PCB基板レイアウトを詰めて100x190mm→100x132mmに縮小、操作パネル配置を変更
均一グリッド配置だった基板を各部品の実パッド範囲に応じて詰め直し、独自A*
グリッドルーターで全結線を再配線(DRCエラー0件・未配線0件を維持)。
VR1/VR2を上部に並べてLEDを間に配置し、SW1を最下部に移動。3Dレンダリング
用にCherry MXスイッチ・ロータリーポットの簡易プレースホルダーも追加。

Co-Authored-By: Claude Sonnet 5 <noreply@anthropic.com>
Parts:
- BT1: footprint (none) -> Connector_PinHeader_2.54mm:PinHeader_1x02_P2.54mm_Vertical; Notes 9V角形電池(006P). footprint: 電池スナップ(基板外配線, 例 Keystone 232)を使用。基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 -> 9V角形電池(006P)。footprint: 電池スナップ(Keystone 232等)のリード線を直接ハンダ付けす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
- J1: footprint (none) -> Connector_Audio:Jack_6.35mm_Neutrik_NRJ6HF_Horizontal; Notes 6.3mmフォンジャック。判断: リング接点(R)を電池(-)の帰路として使用し、モノラルTSプラグのスリーブがリング-スリーブ間を物理的に橋絡した時のみ電池が通電するバッテリーセーブ回路として解釈(標準的なDIYストンプボックス電池スイッチ手法)。footprint: 汎用6.3mmフォンジャック(例 Cliff FCR1295, Lumberg KLB3)。標準ライブラリに完全一致フットプリント無し -> 6.3mmフォンジャック。判断: リング接点(R)を電池(-)の帰路として使用し、モノラルTSプラグのスリーブがリング-スリーブ間を物理的に橋絡した時のみ電池が通電するバッテリーセーブ回路として解釈(標準的なDIYストンプボックス電池スイッチ手法)。footprint: Neutrik NRJ6HF(6.35mm横型TRSジャック)を採用。フットプリントにはTN/RN/SNのスイッチ接点パッドも存在するが本設計では未使用(ネット未接続のまま)
- J2: footprint (none) -> Connector_Audio:Jack_6.35mm_Neutrik_NMJ4HCD2_Horizontal; Notes footprint: 汎用6.3mmフォンジャック(スイッチ無し, 出力専用)。標準ライブラリに完全一致フットプリント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 -> footprint: Neutrik NMJ4HCD2(6.35mm横型モノTSジャック, スイッチ接点TN/SNは未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
- RL1: footprint (none) -> Relay_THT:Relay_DPDT_Schrack-RT2-FormC_RM5mm; Notes 941H-2C-5D (秋月, 5V DPDT)。circuit_reference.md改訂(2026-07-01)によりDPDT両極を使用する真のトゥルーバイパス構成に変更。Pole1(入力切替): 11=COM(J1後段入力信号 IN_SIGNAL), 12=NC接点→DRY(バイパス直通ノード), 14=NO接点→WET_IN(C_inへ、コンプレッサー回路入力)。Pole2(出力切替): 21=COM(J2への出力信号 OUT_SIGNAL), 22=NC接点→DRY(Pole1のNCと共通、バイパス直通ノード), 24=NO接点→WET_OUT(C5後段、コンプレッサー回路出力)。非励磁(バイパス)時は入力→12→DRY→22→出力のみが導通し、励磁時は入力→14→WET_IN→(コンプレッサー回路)→WET_OUT→24→出力のみが導通する真のトゥルーバイパス。footprint: 941H-2C-5Dの標準ライブラリ完全一致フットプリント無し -> 941H-2C-5D (秋月, 5V DPDT)。circuit_reference.md改訂(2026-07-01)によりDPDT両極を使用する真のトゥルーバイパス構成に変更。Pole1(入力切替): 11=COM(J1後段入力信号 IN_SIGNAL), 12=NC接点→DRY(バイパス直通ノード), 14=NO接点→WET_IN(C_inへ、コンプレッサー回路入力)。Pole2(出力切替): 21=COM(J2への出力信号 OUT_SIGNAL), 22=NC接点→DRY(Pole1のNCと共通、バイパス直通ノード), 24=NO接点→WET_OUT(C5後段、コンプレッサー回路出力)。非励磁(バイパス)時は入力→12→DRY→22→出力のみが導通し、励磁時は入力→14→WET_IN→(コンプレッサー回路)→WET_OUT→24→出力のみが導通する真のトゥルーバイパス。footprint: Relay_DPDT_Schrack-RT2-FormC_RM5mm を代用(ピン配置11/12/14/21/22/24/A1/A2はEN50005標準で941H-2C-5Dと一致するはずだが、外形寸法・ピン間隔は941H-2C-5D実物と完全一致しない可能性あり。基板発注前に実物のデータシート寸法図で要確認)
- SW1: footprint (none) -> Button_Switch_Keyboard:SW_Cherry_MX_1.00u_PCB; Notes footprint: Cherry MX PCBマウント(標準ライブラリに完全一致フットプリント無し。5pin中2pi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 -> footprint: Cherry MX 1.00u PCB用footprint(5pinのうちスイッチ接点2pinの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
Changed lines of the file:
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@@
 		(property "Reference" "BT1" (at 22.32 14.32 0) (effects (font (size 1.27 1.27))))
 		(property "Value" "9V" (at 22.32 26.32 0) (effects (font (size 1.27 1.27))))
-		(property "Footprint" "" (at 20.32 20.32 0) (effects (font (size 1.27 1.27)) (hide yes)))
+		(property "Footprint" "Connector_PinHeader_2.54mm:PinHeader_1x02_P2.54mm_Vertical" (at 20.32 20.32 0) (effects (font (size 1.27 1.27)) (hide yes)))
 		(property "Datasheet" "" (at 20.32 20.32 0) (effects (font (size 1.27 1.27)) (hide yes)))
-		(property "Notes" "9V角形電池(006P). footprint: 電池スナップ(基板外配線, 例 Keystone 232)を使用。基板上フットプリント無し" (at 20.32 20.32 0) (effects (font (size 1.27 1.27)) (hide yes)))
+		(property "Notes" "9V角形電池(006P)。footprint: 電池スナップ(Keystone 232等)のリード線を直接ハンダ付けする2Pピンヘッダー相当ランドのプレースホルダー。実際は電池スナップの赤黒リード線をこの2パッドに直接ハンダ付けする想定" (at 20.32 20.32 0) (effects (font (size 1.27 1.27)) (hide yes)))
 		(pin "1")
 		(pin "2")
@@
 		(property "Reference" "J1" (at 22.32 84.17 0) (effects (font (size 1.27 1.27))))
 		(property "Value" "6.3mm TRS(mono use)" (at 22.32 96.17 0) (effects (font (size 1.27 1.27))))
-		(property "Footprint" "" (at 20.32 90.17 0) (effects (font (size 1.27 1.27)) (hide yes)))
+		(property "Footprint" "Connector_Audio:Jack_6.35mm_Neutrik_NRJ6HF_Horizontal" (at 20.32 90.17 0) (effects (font (size 1.27 1.27)) (hide yes)))
 		(property "Datasheet" "" (at 20.32 90.17 0) (effects (font (size 1.27 1.27)) (hide yes)))
-		(property "Notes" "6.3mmフォンジャック。判断: リング接点(R)を電池(-)の帰路として使用し、モノラルTSプラグのスリーブがリング-スリーブ間を物理的に橋絡した時のみ電池が通電するバッテリーセーブ回路として解釈(標準的なDIYストンプボックス電池スイッチ手法)。footprint: 汎用6.3mmフォンジャック(例 Cliff FCR1295, Lumberg KLB3)。標準ライブラリに完全一致フットプリント無し" (at 20.32 90.17 0) (effects (font (size 1.27 1.27)) (hide yes)))
+		(property "Notes" "6.3mmフォンジャック。判断: リング接点(R)を電池(-)の帰路として使用し、モノラルTSプラグのスリーブがリング-スリーブ間を物理的に橋絡した時のみ電池が通電するバッテリーセーブ回路として解釈(標準的なDIYストンプボックス電池スイッチ手法)。footprint: Neutrik NRJ6HF(6.35mm横型TRSジャック)を採用。フットプリントにはTN/RN/SNのスイッチ接点パッドも存在するが本設計では未使用(ネット未接続のまま)" (at 20.32 90.17 0) (effects (font (size 1.27 1.27)) (hide yes)))
 		(pin "T")
 		(pin "S")
@@
 		(property "Reference" "J2" (at 531.59 84.17 0) (effects (font (size 1.27 1.27))))
 		(property "Value" "6.3mm TS(out)" (at 531.59 96.17 0) (effects (font (size 1.27 1.27))))
-		(property "Footprint" "" (at 529.59 90.17 0) (effects (font (size 1.27 1.27)) (hide yes)))
+		(property "Footprint" "Connector_Audio:Jack_6.35mm_Neutrik_NMJ4HCD2_Horizontal" (at 529.59 90.17 0) (effects (font (size 1.27 1.27)) (hide yes)))
 		(property "Datasheet" "" (at 529.59 90.17 0) (effects (font (size 1.27 1.27)) (hide yes)))
-		(property "Notes" "footprint: 汎用6.3mmフォンジャック(スイッチ無し, 出力専用)。標準ライブラリに完全一致フットプリント無し" (at 529.59 90.17 0) (effects (font (size 1.27 1.27)) (hide yes)))
+		(property "Notes" "footprint: Neutrik NMJ4HCD2(6.35mm横型モノTSジャック, スイッチ接点TN/SNは未使用)を採用" (at 529.59 90.17 0) (effects (font (size 1.27 1.27)) (hide yes)))
 		(pin "T")
 		(pin "S")
@@
 		(property "Reference" "SW1" (at 22.32 254.35 0) (effects (font (size 1.27 1.27))))
 		(property "Value" "Cherry MX (手持ち)" (at 22.32 266.35 0) (effects (font (size 1.27 1.27))))
-		(property "Footprint" "" (at 20.32 260.35 0) (effects (font (size 1.27 1.27)) (hide yes)))
+		(property "Footprint" "Button_Switch_Keyboard:SW_Cherry_MX_1.00u_PCB" (at 20.32 260.35 0) (effects (font (size 1.27 1.27)) (hide yes)))
 		(property "Datasheet" "" (at 20.32 260.35 0) (effects (font (size 1.27 1.27)) (hide yes)))
-		(property "Notes" "footprint: Cherry MX PCBマウント(標準ライブラリに完全一致フットプリント無し。5pin中2pinのみ使用)" (at 20.32 260.35 0) (effects (font (size 1.27 1.27)) (hide yes)))
+		(property "Notes" "footprint: Cherry MX 1.00u PCB用footprint(5pinのうちスイッチ接点2pinのみ回路図でネット割当、残り3pin[プレート固定用+LED用穴]はネット未接続のまま)" (at 20.32 260.35 0) (effects (font (size 1.27 1.27)) (hide yes)))
 		(pin "1")
 		(pin "2")
@@
 		(property "Reference" "RL1" (at 281.4 254.35 0) (effects (font (size 1.27 1.27))))
 		(property "Value" "941H-2C-5D" (at 281.4 266.35 0) (effects (font (size 1.27 1.27))))
-		(property "Footprint" "" (at 279.4 260.35 0) (effects (font (size 1.27 1.27)) (hide yes)))
+		(property "Footprint" "Relay_THT:Relay_DPDT_Schrack-RT2-FormC_RM5mm" (at 279.4 260.35 0) (effects (font (size 1.27 1.27)) (hide yes)))
 		(property "Datasheet" "" (at 279.4 260.35 0) (effects (font (size 1.27 1.27)) (hide yes)))
-		(property "Notes" "941H-2C-5D (秋月, 5V DPDT)。circuit_reference.md改訂(2026-07-01)によりDPDT両極を使用する真のトゥルーバイパス構成に変更。Pole1(入力切替): 11=COM(J1後段入力信号 IN_SIGNAL), 12=NC接点→DRY(バイパス直通ノード), 14=NO接点→WET_IN(C_inへ、コンプレッサー回路入力)。Pole2(出力切替): 21=COM(J2への出力信号 OUT_SIGNAL), 22=NC接点→DRY(Pole1のNCと共通、バイパス直通ノード), 24=NO接点→WET_OUT(C5後段、コンプレッサー回路出力)。非励磁(バイパス)時は入力→12→DRY→22→出力のみが導通し、励磁時は入力→14→WET_IN→(コンプレッサー回路)→WET_OUT→24→出力のみが導通する真のトゥルーバイパス。footprint: 941H-2C-5Dの標準ライブラリ完全一致フットプリント無し" (at 279.4 260.35 0) (effects (font (size 1.27 1.27)) (hide yes)))
+		(property "Notes" "941H-2C-5D (秋月, 5V DPDT)。circuit_reference.md改訂(2026-07-01)によりDPDT両極を使用する真のトゥルーバイパス構成に変更。Pole1(入力切替): 11=COM(J1後段入力信号 IN_SIGNAL), 12=NC接点→DRY(バイパス直通ノード), 14=NO接点→WET_IN(C_inへ、コンプレッサー回路入力)。Pole2(出力切替): 21=COM(J2への出力信号 OUT_SIGNAL), 22=NC接点→DRY(Pole1のNCと共通、バイパス直通ノード), 24=NO接点→WET_OUT(C5後段、コンプレッサー回路出力)。非励磁(バイパス)時は入力→12→DRY→22→出力のみが導通し、励磁時は入力→14→WET_IN→(コンプレッサー回路)→WET_OUT→24→出力のみが導通する真のトゥルーバイパス。footprint: Relay_DPDT_Schrack-RT2-FormC_RM5mm を代用(ピン配置11/12/14/21/22/24/A1/A2はEN50005標準で941H-2C-5Dと一致するはずだが、外形寸法・ピン間隔は941H-2C-5D実物と完全一致しない可能性あり。基板発注前に実物のデータシート寸法図で要確認)" (at 279.4 260.35 0) (effects (font (size 1.27 1.27)) (hide yes)))
 		(pin "A1")
 		(pin "A2")
