File: kicad/bass_compressor/bass_compressor.kicad_sch (KiCad schematic)
At the start: 47 parts, among them IC1 LM13700, IC3 TC4013BP, J1 6.3mm TRS(mono use), J2 6.3mm TS(out), Q1 2SC1815, Q2 2SC1815, SW1 Cherry MX (手持ち), U1 TL072

Commit message: PCB出力
Parts:
- C10, C11, C2, C3, C4, C5, C8, C9: footprint Capacitor_THT:C_Radial_D5.0mm_H11.0mm_P2.00mm -> Capacitor_THT:C_Radial_D5.0mm_H11.0mm_P5.00mm
- IC1: value LM13700 -> NJM13700D
- J1: footprint Connector_Audio:Jack_6.35mm_Neutrik_NRJ6HF_Horizontal -> Connector_Audio:Jack_6.35mm_CUI-SameSky_SJ-63053A_Horizontal; Notes 6.3mmフォンジャック。判断: リング接点(R)を電池(-)の帰路として使用し、モノラルTSプラグのスリーブがリング-スリーブ間を物理的に橋絡した時のみ電池が通電するバッテリーセーブ回路として解釈(標準的なDIYストンプボックス電池スイッチ手法)。footprint: Neutrik NRJ6HF(6.35mm横型TRSジャック)を採用。フットプリントにはTN/RN/SNのスイッチ接点パッドも存在するが本設計では未使用(ネット未接続のまま) -> 6.3mmフォンジャック。判断: リング接点(R)を電池(-)の帰路として使用し、モノラルTSプラグのスリーブがリング-スリーブ間を物理的に橋絡した時のみ電池が通電するバッテリーセーブ回路として解釈(標準的なDIYストンプボックス電池スイッチ手法)。2026-07-02: 調達部品をNeutrik NRJ6HFからCUI/Same Sky SJ-63053A(6.35mm横型TRSジャック、スイッチ接点なし、through-hole/right-angle/threaded with nut)に変更したためfootprintも新規作成し差し替え(信号3ピンT/R/S、ピッチ5.00mm、ドリルø1.00mm(+0.2/-0)、位置決め用非導通ペグ穴ø2.20mm(+0.2/-0)×2)。旧NRJ6HF footprintにあったTN/RN/SNのスイッチ接点パッドはSJ-63053Aには存在しないためfootprintから削除(元々ネット未接続だったため回路的な矛盾なし)。注意: SJ-63053AはDigiKey在庫578個のみのDiscontinued(生産完了)品(2026-07-01時点確認)。本基板1台分の製作には支障ないが、将来の追加生産時は代替品の選定が必要。また3DモデルはSame Sky公式サイト・SnapEDAとも入手できなかったため footprint 側の3Dモデル参照は未設定。ペグ穴の正確な位置はデータシートの寸法図(ベクター図)から完全には一意に特定できなかったため、電気的に重要な信号3ピンの座標(5.00mmピッチ・ø1.00mm)を優先して確定し、ペグ穴位置は妥当な工学的推定値。実装前に現物合わせでの確認を推奨。
- RL1: footprint Relay_THT:Relay_DPDT_Schrack-RT2-FormC_RM5mm -> Relay_THT:Relay_DPDT_HsinDa_941H-2C-5D; Notes 941H-2C-5D (秋月, 5V DPDT)。circuit_reference.md改訂(2026-07-01)によりDPDT両極を使用する真のトゥルーバイパス構成に変更。Pole1(入力切替): 11=COM(J1後段入力信号 IN_SIGNAL), 12=NC接点→DRY(バイパス直通ノード), 14=NO接点→WET_IN(C_inへ、コンプレッサー回路入力)。Pole2(出力切替): 21=COM(J2への出力信号 OUT_SIGNAL), 22=NC接点→DRY(Pole1のNCと共通、バイパス直通ノード), 24=NO接点→WET_OUT(C5後段、コンプレッサー回路出力)。非励磁(バイパス)時は入力→12→DRY→22→出力のみが導通し、励磁時は入力→14→WET_IN→(コンプレッサー回路)→WET_OUT→24→出力のみが導通する真のトゥルーバイパス。footprint: Relay_DPDT_Schrack-RT2-FormC_RM5mm を代用(ピン配置11/12/14/21/22/24/A1/A2はEN50005標準で941H-2C-5Dと一致するはずだが、外形寸法・ピン間隔は941H-2C-5D実物と完全一致しない可能性あり。基板発注前に実物のデータシート寸法図で要確認) -> 941H-2C-5D (秋月, 5V DPDT)。circuit_reference.md改訂(2026-07-01)によりDPDT両極を使用する真のトゥルーバイパス構成に変更。Pole1(入力切替): 11=COM(J1後段入力信号 IN_SIGNAL), 12=NC接点→DRY(バイパス直通ノード), 14=NO接点→WET_IN(C_inへ、コンプレッサー回路入力)。Pole2(出力切替): 21=COM(J2への出力信号 OUT_SIGNAL), 22=NC接点→DRY(Pole1のNCと共通、バイパス直通ノード), 24=NO接点→WET_OUT(C5後段、コンプレッサー回路出力)。非励磁(バイパス)時は入力→12→DRY→22→出力のみが導通し、励磁時は入力→14→WET_IN→(コンプレッサー回路)→WET_OUT→24→出力のみが導通する真のトゥルーバイパス。footprint: 2026-07-02にHSINDA公式データシート(941H-2C-5D.pdf p.18 Drilling Plan/Internal Connections)を確認し、footprintをRelay_DPDT_Schrack-RT2-FormC_RM5mm(列ピッチ15.26/20.30/25.34mm・行7.5mm・ドリル1.3mmで実物と不一致)から実寸に合わせて修正(物理ピン1/16=コイルA1/A2、4/13=12/22(NC,DRY)、6/11=11/21(COM)、8/9=14/24(NO・WET)、列ピッチ7.62/12.70/17.78mm、行7.62mm、ドリル0.8mm)。KiCad標準ライブラリに完全一致するfootprintは無かったため、既存footprintを直接編集する形で対応(footprint名はRelay_DPDT_HsinDa_941H-2C-5Dにリネームしたローカル定義)。
Connections:
- net U1B_OUT is gone; now on net U1B_INN: C4.1, R7.2, U1.7
- net WET_IN is gone; now on net DRY: C8.1, RL1.14
